File: Hardware/RotoPDPro.kicad_pcb (KiCad board)
At the start: 2 copper layers, 24.4 x 35.8 mm, 49 parts, among them J1 USB4105-GF-A-060, J2 QWIIC, J3 Screw_Terminal_5mm, J4 Conn_01x08, Q1 RUM001L02T2CL, U1 LM74502DDFR, U2 LMR51635YDDCR, U3 XRS40N10D, U4 INA238, U5 AP33772S, U6 XRS40N10D, U7 TXS0102DCUR

Commit message: V1.2 Release
Parts:
- added C15: 100n, Capacitor_SMD:C_0402_1005Metric, F.Cu at (75.5, 45.5)
- J1: value USB4105-GF-A-060 -> U263-163N-4GS1735
- R5: value 10k -> 20k
Connections:
- U4 pad 8: /VOUT -> /VBUS
Routing:
- net /VBUS: track 19.7 -> 24.0 mm
- net /VOUT: track 12.8 -> 9.91 mm
- net GND: vias 59 -> 60
Other:
- board text added: "RotoPD Rev1.2 4.5V-48V 5A Max USB PD 3.1"
- board text removed: "OUT"
- board text removed: "RotoPD Rev1.1 4.5V-48V 5A Max USB PD 3.1"
Changed lines of the file:
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@@
 			)
 		)
-		(property "LCSC" ""
+		(property "LCSC" "C50314150"
 			(at 0 0 270)
 			(unlocked yes)
@@
 			)
 		)
-		(property "LCSC" ""
+		(property "LCSC" "C50314150"
 			(at 0 0 90)
 			(unlocked yes)
@@
 			)
 		)
-		(property "LCSC" ""
+		(property "LCSC" "C2868250"
 			(at 0 0 0)
 			(unlocked yes)
@@
 			(layers "F.Cu" "F.Mask" "F.Paste")
 			(roundrect_rratio 0.25)
-			(net 9 "/VOUT")
+			(net 10 "/VBUS")
 			(pinfunction "Vbus")
 			(pintype "input")
@@
 	(footprint "Capacitor_SMD:C_0402_1005Metric"
 		(layer "F.Cu")
+		(at 75.461 45.469)
+		(descr "Capacitor SMD 0402 (1005 Metric), square (rectangular) end terminal, IPC-7351 nominal, (Body size source: IPC-SM-782 page 76, https://www.pcb-3d.com/wordpress/wp-content/uploads/ipc-sm-782a_amendment_1_and_2.pdf), generated with kicad-footprint-generator")
+		(tags "capacitor")
+		(property "Reference" "C15"
+			(at 0 -1.16 0)
+			(layer "F.SilkS")
+			(hide yes)
+			(effects
+				(font
+					(size 1 1)
+					(thickness 0.15)
+				)
+			)
+		)
+		(property "Value" "100n"
+			(at 0 1.16 0)
+			(layer "F.Fab")
+			(effects
+				(font
+					(size 1 1)
+					(thickness 0.15)
+				)
+			)
+		)
+		(property "Datasheet" "~"
+			(at 0 0 0)
+			(layer "F.Fab")
+			(hide yes)
+			(effects
+				(font
+					(size 1.27 1.27)
+					(thickness 0.15)
+				)
+			)
+		)
+		(property "Description" ""
+			(at 0 0 0)
+			(layer "F.Fab")
+			(hide yes)
+			(effects
+				(font
+					(size 1.27 1.27)
+					(thickness 0.15)
+				)
+			)
+		)
+		(property "LCSC" "C162179"
+			(at 0 0 0)
+			(unlocked yes)
+			(layer "F.Fab")
+			(hide yes)
+			(effects
+				(font
+					(size 1 1)
+					(thickness 0.15)
+				)
+			)
+		)
+		(property ki_fp_filters "C_*")
+		(sheetname "/")
+		(sheetfile "RotoPDPro.kicad_sch")
+		(attr smd)
+		(fp_line
+			(start -0.107836 -0.36)
+			(end 0.107836 -0.36)
+			(stroke
+				(width 0.12)
+				(type solid)
+			)
+			(layer "F.SilkS")
+		)
+		(fp_line
+			(start -0.107836 0.36)
+			(end 0.107836 0.36)
+			(stroke
+				(width 0.12)
+				(type solid)
+			)
+			(layer "F.SilkS")
+		)
+		(fp_rect
+			(start -0.91 -0.46)
+			(end 0.91 0.46)
+			(stroke
+				(width 0.05)
+				(type solid)
+			)
+			(fill no)
+			(layer "F.CrtYd")
+		)
+		(fp_rect
+			(start -0.5 -0.25)
+			(end 0.5 0.25)
+			(stroke
+				(width 0.1)
+				(type solid)
+			)
+			(fill no)
+			(layer "F.Fab")
+		)
+		(fp_text user "${REFERENCE}"
+			(at 0 0 0)
+			(layer "F.Fab")
+			(effects
+				(font
+					(size 0.25 0.25)
+					(thickness 0.04)
+				)
+			)
+		)
+		(pad "1" smd roundrect
+			(at -0.48 0)
+			(size 0.56 0.62)
+			(layers "F.Cu" "F.Mask" "F.Paste")
+			(roundrect_rratio 0.25)
+			(net 10 "/VBUS")
+			(pintype "passive")
+		)
+		(pad "2" smd roundrect
+			(at 0.48 0)
+			(size 0.56 0.62)
+			(layers "F.Cu" "F.Mask" "F.Paste")
+			(roundrect_rratio 0.25)
+			(net 2 "GND")
+			(pintype "passive")
+		)
+		(embedded_fonts no)
+		(model "${KICAD9_3DMODEL_DIR}/Capacitor_SMD.3dshapes/C_0402_1005Metric.step"
+			(offset
+				(xyz 0 0 0)
+			)
+			(scale
+				(xyz 1 1 1)
+			)
+			(rotate
+				(xyz 0 0 0)
+			)
+		)
+	)
+	(footprint "Capacitor_SMD:C_0402_1005Metric"
+		(layer "F.Cu")
 		(at 73.461 44.269 180)
 		(descr "Capacitor SMD 0402 (1005 Metric), square (rectangular) end terminal, IPC-7351 nominal, (Body size source: IPC-SM-782 page 76, https://www.pcb-3d.com/wordpress/wp-content/uploads/ipc-sm-782a_amendment_1_and_2.pdf), generated with kicad-footprint-generator")
@@
 			)
 		)
-		(property "LCSC" ""
+		(property "LCSC" "C5219202"
 			(at 0 0 0)
 			(unlocked yes)
@@
 			)
 		)
-		(property "LCSC" ""
+		(property "LCSC" "C138714"
 			(at 0 0 90)
 			(unlocked yes)
@@
 			)
 		)
-		(property "LCSC2" ""
+		(property "LCSC2" "C2827646"
 			(at 0 0 90)
 			(unlocked yes)
@@
 			)
 		)
-		(property "LCSC" ""
+		(property "LCSC" "C5349682"
 			(at 0 0 180)
 			(unlocked yes)
@@
 			)
 		)
-		(property "Value" "10k"
+		(property "Value" "20k"
 			(at 0 1.43 90)
 			(layer "F.Fab")
@@
 			)
 		)
-		(property "LCSC" ""
+		(property "LCSC" "C24374260"
 			(at 0 0 180)
 			(unlocked yes)
@@
 			)
 		)
-		(property "LCSC" ""
+		(property "LCSC" "C53434"
 			(at 0 0 90)
 			(unlocked yes)
@@
 			)
 		)
-		(property "Value" "USB4105-GF-A-060"
+		(property "Value" "U263-163N-4GS1735"
 			(at 0 -2.65 180)
 			(unlocked yes)
@@
 			)
 		)
-		(property "LCSC" ""
+		(property "LCSC" "C2931470"
 			(at 0 0 180)
 			(unlocked yes)
@@
 			)
 		)
-		(property "LCSC" ""
+		(property "LCSC" "C253528"
 			(at 0 0 180)
 			(unlocked yes)
@@
 			)
 		)
-		(property "LCSC Part" ""
+		(property "LCSC Part" "C45262770"
 			(at 0 0 270)
 			(unlocked yes)
@@
 		)
 	)
-	(gr_text "OUT"
-		(at 65.761 68.669 90)
-		(layer "F.SilkS")
-		(effects
-			(font
-				(size 0.85 0.85)
-				(thickness 0.17)
-				(bold yes)
-			)
-			(justify left bottom)
-		)
-	)
 	(gr_text "SDA"
 		(at 62.961 47.269 0)
@@
 		)
 	)
-	(gr_text "RotoPD       Rev1.1\n4.5V-48V 5A Max\nUSB PD 3.1"
+	(gr_text "RotoPD       Rev1.2\n4.5V-48V 5A Max\nUSB PD 3.1"
 		(at 79.761 59.969 0)
 		(layer "B.SilkS")
@@
 	)
 	(via
+		(at 75.961 46.169)
+		(size 0.45)
+		(drill 0.2)
+		(layers "F.Cu" "B.Cu")
+		(free yes)
+		(net 2)
+	)
+	(via
 		(at 74.661 60.569)
 		(size 0.45)
@@
 	)
 	(segment
-		(start 77.511 49.219)
-		(end 76.961 48.669)
-		(width 0.15)
-		(layer "F.Cu")
-		(net 9)
-	)
-	(segment
 		(start 77.711 48.819)
 		(end 77.561 48.819)
@@
 	)
 	(segment
-		(start 76.511 47.769)
-		(end 75.711 47.769)
-		(width 0.15)
-		(layer "F.Cu")
-		(net 9)
-	)
-	(segment
-		(start 76.961 48.219)
-		(end 76.511 47.769)
-		(width 0.15)
-		(layer "F.Cu")
-		(net 9)
-	)
-	(segment
 		(start 69.686 65.869)
 		(end 75.261 65.869)
@@
 	)
 	(segment
-		(start 77.711 49.219)
-		(end 77.511 49.219)
-		(width 0.15)
-		(layer "F.Cu")
-		(net 9)
-	)
-	(segment
 		(start 77.561 48.819)
 		(end 77.311 48.569)
@@
 	)
 	(segment
-		(start 76.961 48.669)
-		(end 76.961 48.219)
-		(width 0.15)
-		(layer "F.Cu")
-		(net 9)
-	)
-	(segment
 		(start 72.981 44.269)
 		(end 72.0935 44.269)
@@
 	)
 	(segment
+		(start 74.461 47.469)
+		(end 74.461 45.989)
+		(width 0.15)
+		(layer "F.Cu")
+		(net 10)
+	)
+	(segment
 		(start 75.461 43.069)
 		(end 74.761 43.769)
@@
 	(segment
 		(start 73.261 49.769)
-		(end 73.261 46.169)
+		(end 73.261 47.769)
 		(width 0.5)
 		(layer "F.Cu")
@@
 	)
 	(segment
+		(start 75.711 47.769)
+		(end 74.761 47.769)
+		(width 0.15)
+		(layer "F.Cu")
+		(net 10)
+	)
+	(segment
+		(start 74.461 45.989)
+		(end 74.981 45.469)
+		(width 0.15)
+		(layer "F.Cu")
+		(net 10)
+	)
+	(segment
 		(start 73.6985 43.5515)
 		(end 72.981 44.269)
@@
 	)
 	(segment
+		(start 73.261 47.769)
+		(end 73.261 46.169)
+		(width 0.5)
+		(layer "F.Cu")
+		(net 10)
+	)
+	(segment
+		(start 74.961 45.469)
+		(end 74.461 44.969)
+		(width 0.15)
+		(layer "F.Cu")
+		(net 10)
+	)
+	(segment
 		(start 73.161 49.869)
 		(end 73.261 49.769)
@@
 	)
 	(segment
+		(start 74.461 44.969)
+		(end 74.761 44.669)
+		(width 0.5)
+		(layer "F.Cu")
+		(net 10)
+	)
+	(segment
 		(start 75.561 43.069)
 		(end 75.461 43.069)
@@
 	)
 	(segment
+		(start 74.761 47.769)
+		(end 74.461 47.469)
+		(width 0.15)
+		(layer "F.Cu")
+		(net 10)
+	)
+	(segment
 		(start 73.6985 43.144)
 		(end 74.136 43.144)
@@
 	)
 	(segment
+		(start 74.981 45.469)
+		(end 74.961 45.469)
+		(width 0.15)
+		(layer "F.Cu")
+		(net 10)
+	)
+	(segment
 		(start 73.261 46.169)
-		(end 74.761 44.669)
+		(end 74.461 44.969)
 		(width 0.5)
 		(layer "F.Cu")
