File: Hardware/RotoPDPro.kicad_sch (KiCad schematic)
At the start: 48 parts, among them J1 USB4105-GF-A-060, J2 QWIIC, J3 Screw_Terminal_5mm, J4 Conn_01x08, Q1 RUM001L02T2CL, U1 LM74502DDFR, U2 LMR51635YDDCR, U3 XRS40N10D, U4 INA238, U5 AP33772S, U6 XRS40N10D, U7 TXS0102DCUR

Commit message: V1.2 Release
Parts:
- added C15: 100n, Capacitor_SMD:C_0402_1005Metric, symbol Device:C
- D4: LCSC (none) -> C138714; LCSC2 (none) -> C2827646
- J1: value USB4105-GF-A-060 -> U263-163N-4GS1735; LCSC (none) -> C2931470
- L1: LCSC (none) -> C5349682
- Q1: LCSC (none) -> C253528
- R5: value 10k -> 20k
- U1: LCSC (none) -> C5219202
- U2: LCSC Part (none) -> C45262770
- U3, U6: LCSC (none) -> C50314150
- U4: LCSC (none) -> C2868250
- U5: LCSC (none) -> C24374260
- U7: LCSC (none) -> C53434
Connections:
- net GND: now also C15.2
- net VBUS: now also U4.8 (Vbus), C15.1
- net VOUT: no longer U4.8 (Vbus)
Changed lines of the file:
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@@
 	(title_block
 		(title "RotoPD Pro")
-		(date "2026-02-07")
-		(rev "V1.1")
+		(date "2026-08-09")
+		(rev "V1.2")
 		(company "CentyLab")
 	)
@@
 	)
 	(junction
+		(at 96.52 29.21)
+		(diameter 0)
+		(color 0 0 0 0)
+	)
+	(junction
 		(at 186.69 50.8)
 		(diameter 0)
@@
 	)
 	(junction
-		(at 147.32 29.21)
-		(diameter 0)
-		(color 0 0 0 0)
-	)
-	(junction
 		(at 78.74 162.56)
 		(diameter 0)
@@
 	)
 	(junction
+		(at 147.32 33.02)
+		(diameter 0)
+		(color 0 0 0 0)
+	)
+	(junction
 		(at 91.44 63.5)
 		(diameter 0)
@@
 	(wire
 		(pts
-			(xy 147.32 29.21) (xy 147.32 50.8)
+			(xy 148.59 50.8) (xy 147.32 50.8)
 		)
 		(stroke
@@
 	(wire
 		(pts
-			(xy 148.59 50.8) (xy 147.32 50.8)
+			(xy 304.8 133.35) (xy 307.34 133.35)
 		)
 		(stroke
@@
 	(wire
 		(pts
-			(xy 304.8 133.35) (xy 307.34 133.35)
+			(xy 323.85 44.45) (xy 336.55 44.45)
 		)
 		(stroke
@@
 	(wire
 		(pts
-			(xy 323.85 44.45) (xy 336.55 44.45)
+			(xy 218.44 111.76) (xy 262.89 111.76)
 		)
 		(stroke
@@
 	(wire
 		(pts
-			(xy 218.44 111.76) (xy 262.89 111.76)
+			(xy 72.39 168.91) (xy 86.36 168.91)
 		)
 		(stroke
@@
 	(wire
 		(pts
-			(xy 72.39 168.91) (xy 86.36 168.91)
+			(xy 151.13 40.64) (xy 151.13 41.91)
 		)
 		(stroke
@@
 	(wire
 		(pts
+			(xy 147.32 33.02) (xy 147.32 19.05)
+		)
+		(stroke
+			(width 0)
+			(type default)
+		)
+	)
+	(wire
+		(pts
 			(xy 251.46 123.19) (xy 251.46 115.57)
 		)
@@
 	(wire
 		(pts
-			(xy 93.98 29.21) (xy 99.06 29.21)
+			(xy 93.98 29.21) (xy 96.52 29.21)
 		)
 		(stroke
@@
 	(wire
 		(pts
-			(xy 147.32 29.21) (xy 200.66 29.21)
+			(xy 147.32 19.05) (xy 96.52 19.05)
 		)
 		(stroke
@@
 	(wire
 		(pts
+			(xy 147.32 50.8) (xy 147.32 33.02)
+		)
+		(stroke
+			(width 0)
+			(type default)
+		)
+	)
+	(wire
+		(pts
 			(xy 91.44 55.88) (xy 93.98 55.88)
 		)
@@
 	(wire
 		(pts
-			(xy 143.51 29.21) (xy 147.32 29.21)
+			(xy 147.32 33.02) (xy 151.13 33.02)
+		)
+		(stroke
+			(width 0)
+			(type default)
+		)
+	)
+	(wire
+		(pts
+			(xy 143.51 29.21) (xy 200.66 29.21)
 		)
 		(stroke
@@
 	(wire
 		(pts
+			(xy 96.52 29.21) (xy 99.06 29.21)
+		)
+		(stroke
+			(width 0)
+			(type default)
+		)
+	)
+	(wire
+		(pts
+			(xy 96.52 19.05) (xy 96.52 29.21)
+		)
+		(stroke
+			(width 0)
+			(type default)
+		)
+	)
+	(wire
+		(pts
 			(xy 200.66 29.21) (xy 212.09 29.21)
 		)
@@
 			)
 		)
-		(property "LCSC" ""
+		(property "LCSC" "C24374260"
 			(at 205.74 123.19 0)
 			(effects
@@
 			)
 		)
-		(property "LCSC" ""
+		(property "LCSC" "C50314150"
 			(at 104.14 29.21 0)
 			(effects
@@
 			)
 		)
-		(property "LCSC" ""
+		(property "LCSC" "C5349682"
 			(at 91.44 162.56 90)
 			(effects
@@
 			)
 		)
-		(property "LCSC" ""
+		(property "LCSC" "C138714"
 			(at 49.53 105.41 0)
 			(effects
@@
 			)
 		)
-		(property "LCSC2" ""
+		(property "LCSC2" "C2827646"
 			(at 49.53 105.41 0)
 			(effects
@@
 			)
 		)
-		(property "Value" "USB4105-GF-A-060"
+		(property "Value" "U263-163N-4GS1735"
 			(at 30.48 24.13 0)
 			(effects
@@
 			)
 		)
-		(property "LCSC" ""
+		(property "LCSC" "C2931470"
 			(at 30.48 44.45 0)
 			(effects
@@
 	)
 	(symbol
+		(lib_id "Device:C")
+		(at 151.13 36.83 0)
+		(unit 1)
+		(exclude_from_sim no)
+		(in_bom yes)
+		(on_board yes)
+		(dnp no)
+		(property "Reference" "C15"
+			(at 153.67 35.56 0)
+			(effects
+				(font
+					(size 1.27 1.27)
+				)
+				(justify left)
+			)
+		)
+		(property "Value" "100n"
+			(at 153.67 38.1 0)
+			(effects
+				(font
+					(size 1.27 1.27)
+				)
+				(justify left)
+			)
+		)
+		(property "Footprint" "Capacitor_SMD:C_0402_1005Metric"
+			(at 152.0952 40.64 0)
+			(effects
+				(font
+					(size 1.27 1.27)
+				)
+				(hide yes)
+			)
+		)
+		(property "Datasheet" "~"
+			(at 151.13 36.83 0)
+			(effects
+				(font
+					(size 1.27 1.27)
+				)
+				(hide yes)
+			)
+		)
+		(property "Description" ""
+			(at 151.13 36.83 0)
+			(effects
+				(font
+					(size 1.27 1.27)
+				)
+				(hide yes)
+			)
+		)
+		(property "LCSC" "C162179"
+			(at 151.13 36.83 0)
+			(effects
+				(font
+					(size 1.27 1.27)
+				)
+				(hide yes)
+			)
+		)
+		(pin "1"
+		)
+		(pin "2"
+		)
+		(instances
+			(project "RotoPDPro"
+				(path "/1ee0bb08-61c0-4e99-ad63-6a3fb775020e"
+					(reference "C15")
+					(unit 1)
+				)
+			)
+		)
+	)
+	(symbol
 		(lib_id "Mechanical:MountingHole")
 		(at 199.39 187.96 0)
@@
 			)
 		)
-		(property "LCSC" ""
+		(property "LCSC" "C5219202"
 			(at 110.49 60.96 0)
 			(effects
@@
 	(symbol
 		(lib_id "power:GND")
+		(at 151.13 41.91 0)
+		(mirror y)
+		(unit 1)
+		(exclude_from_sim no)
+		(in_bom yes)
+		(on_board yes)
+		(dnp no)
+		(property "Reference" "#PWR039"
+			(at 151.13 48.26 0)
+			(effects
+				(font
+					(size 1.27 1.27)
+				)
+				(hide yes)
+			)
+		)
+		(property "Value" "GND"
+			(at 151.13 45.974 0)
+			(effects
+				(font
+					(size 1.27 1.27)
+				)
+			)
+		)
+		(property "Footprint" ""
+			(at 151.13 41.91 0)
+			(effects
+				(font
+					(size 1.27 1.27)
+				)
+				(hide yes)
+			)
+		)
+		(property "Datasheet" ""
+			(at 151.13 41.91 0)
+			(effects
+				(font
+					(size 1.27 1.27)
+				)
+				(hide yes)
+			)
+		)
+		(property "Description" "Power symbol creates a global label with name \"GND\" , ground"
+			(at 151.13 41.91 0)
+			(effects
+				(font
+					(size 1.27 1.27)
+				)
+				(hide yes)
+			)
+		)
+		(pin "1"
+		)
+		(instances
+			(project "RotoPDPro"
+				(path "/1ee0bb08-61c0-4e99-ad63-6a3fb775020e"
+					(reference "#PWR039")
+					(unit 1)
+				)
+			)
+		)
+	)
+	(symbol
+		(lib_id "power:GND")
 		(at 102.87 193.04 0)
 		(unit 1)
@@
 			)
 		)
-		(property "LCSC" ""
+		(property "LCSC" "C53434"
 			(at 283.21 50.8 0)
 			(effects
@@
 			)
 		)
-		(property "LCSC" ""
+		(property "LCSC" "C253528"
 			(at 120.65 107.95 0)
 			(effects
@@
 			)
 		)
-		(property "LCSC" ""
+		(property "LCSC" "C50314150"
 			(at 123.19 29.21 0)
 			(effects
@@
 			)
 		)
-		(property "LCSC" ""
+		(property "LCSC" "C2868250"
 			(at 158.75 58.42 0)
 			(effects
@@
 			)
 		)
-		(property "Value" "10k"
+		(property "Value" "20k"
 			(at 203.2 35.5599 0)
 			(effects
@@
 			)
 		)
-		(property "LCSC Part" ""
+		(property "LCSC Part" "C45262770"
 			(at 64.262 177.546 0)
 			(effects
